Commit message: + urdf

File: spotmicro/util/pybullet_data/assets/urdf/spot.urdf (robot description, URDF)
Before this commit: robot , 21 links, 20 joints
Links:
- removed link DC_conv_1
- removed link DC_conv_2
- removed link back_left_down_leg
- removed link back_left_up_leg
- removed link back_right_down_leg
- removed link back_right_up_leg
- removed link bat
- removed link camera
- removed link front_left_down_leg
- removed link front_left_up_leg
- removed link front_right_down_leg
- removed link front_right_up_leg
- removed link jetson
- removed link mcu
- removed link motor_front_left_hip
- removed link ultra_sonic_1
- removed link ultra_sonic_2
- added link back, mass 0.1; collision box size=0.114 0.075 0.085; visual mesh filename=package://mini_ros/stl/OpenQuadruped/Back.stl scale=1 1 1
- added link back_bracket, mass 0.1; collision box size=0.025 0.075 0.085; visual mesh filename=package://mini_ros/stl/OpenQuadruped/Back_Bracket.stl scale=1 1 1
- added link back_left_foot, mass 0.005; collision mesh filename=package://mini_ros/stl/OpenQuadruped/LEFT_FOOT.stl scale=1 1 1; visual mesh filename=package://mini_ros/stl/OpenQuadruped/LEFT_FOOT.stl scale=1 1 1
- added link back_left_lower_leg, mass 0.05; collision box size=0.035 0.035 0.12; visual mesh filename=package://mini_ros/stl/OpenQuadruped/LEFT_LOWER_LEG.stl scale=1 1 1
- added link back_left_upper_leg, mass 0.13; collision box size=0.035 0.035 0.11; visual mesh filename=package://mini_ros/stl/OpenQuadruped/LEFT_UPPER_LEG.stl scale=1 1 1
- added link back_right_foot, mass 0.005; collision mesh filename=package://mini_ros/stl/OpenQuadruped/RIGHT_FOOT.stl scale=1 1 1; visual mesh filename=package://mini_ros/stl/OpenQuadruped/RIGHT_FOOT.stl scale=1 1 1
- added link back_right_lower_leg, mass 0.05; collision box size=0.035 0.035 0.12; visual mesh filename=package://mini_ros/stl/OpenQuadruped/RIGHT_LOWER_LEG.stl scale=1 1 1
- added link back_right_upper_leg, mass 0.13; collision box size=0.035 0.035 0.11; visual mesh filename=package://mini_ros/stl/OpenQuadruped/RIGHT_UPPER_LEG.stl scale=1 1 1
- added link battery, mass 0.4; collision box size=0.048 0.145 0.026; visual mesh filename=package://mini_ros/stl/OpenQuadruped/Battery.stl scale=1 1 1
- added link chassis_left, mass 0.01; collision box size=0.06 0.15 0.006; visual mesh filename=package://mini_ros/stl/OpenQuadruped/Chassis_Left_Side.stl scale=1 1 1
- added link chassis_right, mass 0.01; collision box size=0.06 0.15 0.006; visual mesh filename=package://mini_ros/stl/OpenQuadruped/Chassis_Right_Side.stl scale=1 1 1
- added link front, mass 0.1; collision box size=0.114 0.045 0.085; visual mesh filename=package://mini_ros/stl/OpenQuadruped/Front.stl scale=1 1 1
- added link front_bracket, mass 0.1; collision box size=0.025 0.075 0.085; visual mesh filename=package://mini_ros/stl/OpenQuadruped/Front_Bracket.stl scale=1 1 1
- added link front_left_foot, mass 0.005; collision mesh filename=package://mini_ros/stl/OpenQuadruped/LEFT_FOOT.stl scale=1 1 1; visual mesh filename=package://mini_ros/stl/OpenQuadruped/LEFT_FOOT.stl scale=1 1 1
- added link front_left_hip, mass 0.2; collision box size=0.05 0.065 0.065; visual mesh filename=package://mini_ros/stl/OpenQuadruped/LEFT_HIP.stl scale=1 1 1
- added link front_left_lower_leg, mass 0.05; collision box size=0.035 0.035 0.12; visual mesh filename=package://mini_ros/stl/OpenQuadruped/LEFT_LOWER_LEG.stl scale=1 1 1
- added link front_left_upper_leg, mass 0.13; collision box size=0.035 0.035 0.11; visual mesh filename=package://mini_ros/stl/OpenQuadruped/LEFT_UPPER_LEG.stl scale=1 1 1
- added link front_right_foot, mass 0.005; collision mesh filename=package://mini_ros/stl/OpenQuadruped/RIGHT_FOOT.stl scale=1 1 1; visual mesh filename=package://mini_ros/stl/OpenQuadruped/RIGHT_FOOT.stl scale=1 1 1
- added link front_right_lower_leg, mass 0.05; collision box size=0.035 0.035 0.12; visual mesh filename=package://mini_ros/stl/OpenQuadruped/RIGHT_LOWER_LEG.stl scale=1 1 1
- added link front_right_upper_leg, mass 0.13; collision box size=0.035 0.035 0.11; visual mesh filename=package://mini_ros/stl/OpenQuadruped/RIGHT_UPPER_LEG.stl scale=1 1 1
- link back_left_hip: mass 0.105 -> 0.2; geometry collision box size=0.05 0.065 0.065; visual mesh filename=package://mini_ros/stl/OpenQuadruped/LEFT_HIP.stl scale=1 1 1
- link back_right_hip: mass 0.105 -> 0.2; geometry collision box size=0.05 0.065 0.065; visual mesh filename=package://mini_ros/stl/OpenQuadruped/RIGHT_HIP.stl scale=1 1 1
- link base_link: mass 0.83802 -> 0.6; geometry collision box size=0.114 0.2 0.1; visual mesh filename=package://mini_ros/stl/OpenQuadruped/MAINBODY.stl scale=1 1 1
- link front_right_hip: mass 0.105 -> 0.2; geometry collision box size=0.05 0.065 0.065; visual mesh filename=package://mini_ros/stl/OpenQuadruped/RIGHT_HIP.stl scale=1 1 1
Joints:
- removed joint base_DC_1
- removed joint base_DC_2
- removed joint base_bat
- removed joint base_camera
- removed joint base_jetson
- removed joint base_mcu
- removed joint base_us_1
- removed joint base_us_2
- removed joint front_left_foot
- removed joint front_left_leg
- removed joint front_left_shoulder
- removed joint front_right_foot
- removed joint front_right_leg
- removed joint front_right_shoulder
- removed joint rear_left_foot
- removed joint rear_left_leg
- removed joint rear_left_shoulder
- removed joint rear_right_foot
- removed joint rear_right_leg
- removed joint rear_right_shoulder
- added joint back_left_leg_foot: type fixed, parent back_left_lower_leg, child back_left_foot, origin xyz=0 0 -0.1265 rpy=0 0 0
- added joint back_right_leg_foot: type fixed, parent back_right_lower_leg, child back_right_foot, origin xyz=0 0 -0.1265 rpy=0 0 0
- added joint base_back: type fixed, parent base_link, child back, origin xyz=0 0 0 rpy=0 0 0
- added joint base_back_bracket: type fixed, parent base_link, child back_bracket, origin xyz=0 0 0 rpy=0 0 0
- added joint base_battery: type fixed, parent base_link, child battery, origin xyz=-0.01 0 -0.0225 rpy=0 0 0
- added joint base_front: type fixed, parent base_link, child front, origin xyz=0 0 0 rpy=0 0 0
- added joint base_front_bracket: type fixed, parent base_link, child front_bracket, origin xyz=0 0 0 rpy=0 0 0
- added joint base_left: type fixed, parent base_link, child chassis_left, origin xyz=0.00 0.052 0 rpy=0 0 0
- added joint base_right: type fixed, parent base_link, child chassis_right, origin xyz=0.00 -0.052 0 rpy=0 0 0
- added joint front_left_leg_foot: type fixed, parent front_left_lower_leg, child front_left_foot, origin xyz=0 0 -0.1265 rpy=0 0 0
- added joint front_right_leg_foot: type fixed, parent front_right_lower_leg, child front_right_foot, origin xyz=0 0 -0.1265 rpy=0 0 0
- added joint motor_back_left_hip: type revolute, parent back_bracket, child back_left_hip, origin xyz=-0.1365 0.0394 0.022 rpy=0 0 0, axis 1 0 0, limit lower=-1.04 upper=1.04 effort=1000.0 velocity=0.7
- added joint motor_back_left_lower_leg: type revolute, parent back_left_upper_leg, child back_left_lower_leg, origin xyz=-0.005 0.018 -0.109 rpy=0 0 0, axis 0 1 0, limit lower=-2.9 upper=1.57079632679 effort=1000.0 velocity=0.7
- added joint motor_back_left_upper_leg: type revolute, parent back_left_hip, child back_left_upper_leg, origin xyz=0.0015 0.045 -0.0087 rpy=0 0 0, axis 0 1 0, limit lower=-1.57079632679 upper=2.59 effort=1000.0 velocity=0.7
- added joint motor_back_right_hip: type revolute, parent back_bracket, child back_right_hip, origin xyz=-0.1365 -0.0394 0.022 rpy=0 0 0, axis 1 0 0, limit lower=-1.04 upper=1.04 effort=1000.0 velocity=0.7
- added joint motor_back_right_lower_leg: type revolute, parent back_right_upper_leg, child back_right_lower_leg, origin xyz=-0.005 -0.018 -0.109 rpy=0 0 0, axis 0 1 0, limit lower=-2.9 upper=1.57079632679 effort=1000.0 velocity=0.7
- added joint motor_back_right_upper_leg: type revolute, parent back_right_hip, child back_right_upper_leg, origin xyz=0.0015 -0.045 -0.0087 rpy=0 0 0, axis 0 1 0, limit lower=-1.57079632679 upper=2.59 effort=1000.0 velocity=0.7
- added joint motor_front_left_hip: type revolute, parent front_bracket, child front_left_hip, origin xyz=0.0915 0.0394 0.022 rpy=0 0 0, axis 1 0 0, limit lower=-1.04 upper=1.04 effort=1000.0 velocity=0.7
- added joint motor_front_left_lower_leg: type revolute, parent front_left_upper_leg, child front_left_lower_leg, origin xyz=-0.005 0.018 -0.109 rpy=0 0 0, axis 0 1 0, limit lower=-2.9 upper=1.57079632679 effort=1000.0 velocity=0.7
- added joint motor_front_left_upper_leg: type revolute, parent front_left_hip, child front_left_upper_leg, origin xyz=0.0015 0.045 -0.0087 rpy=0 0 0, axis 0 1 0, limit lower=-1.57079632679 upper=2.59 effort=1000.0 velocity=0.7
- added joint motor_front_right_hip: type revolute, parent front_bracket, child front_right_hip, origin xyz=0.0915 -0.0394 0.022 rpy=0 0 0, axis 1 0 0, limit lower=-1.04 upper=1.04 effort=1000.0 velocity=0.7
- added joint motor_front_right_lower_leg: type revolute, parent front_right_upper_leg, child front_right_lower_leg, origin xyz=-0.005 -0.018 -0.109 rpy=0 0 0, axis 0 1 0, limit lower=-2.9 upper=1.57079632679 effort=1000.0 velocity=0.7
- added joint motor_front_right_upper_leg: type revolute, parent front_right_hip, child front_right_upper_leg, origin xyz=0.0015 -0.045 -0.0087 rpy=0 0 0, axis 0 1 0, limit lower=-1.57079632679 upper=2.59 effort=1000.0 velocity=0.7
