Commit message: fix urdf

File: spotmicro/util/pybullet_data/assets/urdf/spot_cv.urdf (robot description, URDF)
Before this commit: robot , 25 links, 24 joints
Links:
- link back_left_foot_link: mass 0.05 -> 0.01
- link back_right_foot_link: mass 0.05 -> 0.01
- link front_left_foot_link: mass 0.05 -> 0.01
- link front_right_foot_link: mass 0.05 -> 0.01
Joints:
- joint back_left_leg_foot: origin xyz=-0.00525163411775806 -0.0308000000000001 -0.127791974605836 rpy=0 0 0 -> xyz=-0.003621 -0.0308 -0.12839 rpy=0 0 0
- joint back_right_leg_foot: origin xyz=-0.00525006243581849 0.0308 -0.12779266855331 rpy=0 0 0 -> xyz=-0.0052516 0.0308 -0.12779 rpy=0 0 0
- joint front_left_leg_foot: origin xyz=-0.0052516 -0.0308 -0.12779 rpy=0 0 0 -> xyz=-0.003621 -0.0308 -0.12839 rpy=0 0 0
- joint front_right_leg_foot: origin xyz=-0.00454106015218625 0.0308 -0.128081029544538 rpy=0 0 0 -> xyz=-0.0052516 0.0308 -0.12779 rpy=0 0 0
- joint motor_back_left_hip: axis -1 0 0 -> 1 0 0
- joint motor_back_left_lower_leg: axis 0 -1 0 -> 0 1 0; limit lower=-0.1 upper=2.59 effort=1000 velocity=0.5 -> lower=-2.59 upper=0.1 effort=1000 velocity=0.5
- joint motor_back_left_upper_leg: axis 0 -1 0 -> 0 1 0; limit lower=-2.666 upper=1.548 effort=1000 velocity=0.5 -> lower=-1.548 upper=2.666 effort=1000 velocity=0.5
- joint motor_back_right_hip: axis -1 0 0 -> 1 0 0
- joint motor_back_right_lower_leg: axis 0 -1 0 -> 0 1 0; limit lower=-0.1 upper=2.59 effort=1000 velocity=0.5 -> lower=-2.59 upper=0.1 effort=1000 velocity=0.5
- joint motor_back_right_upper_leg: axis 0 -1 0 -> 0 1 0; limit lower=-2.666 upper=1.548 effort=1000 velocity=0.5 -> lower=-1.548 upper=2.666 effort=1000 velocity=0.5
- joint motor_front_left_hip: axis -1 0 0 -> 1 0 0
- joint motor_front_left_lower_leg: axis 0 -1 0 -> 0 1 0; limit lower=-0.1 upper=2.59 effort=1000 velocity=0.5 -> lower=-2.59 upper=0.1 effort=1000 velocity=0.5
- joint motor_front_left_upper_leg: axis 0 -1 0 -> 0 1 0; limit lower=-2.666 upper=1.548 effort=1000 velocity=0.5 -> lower=-1.548 upper=2.666 effort=1000 velocity=0.5
- joint motor_front_right_hip: axis -1 0 0 -> 1 0 0
- joint motor_front_right_lower_leg: axis 0 -1 0 -> 0 1 0; limit lower=-0.1 upper=2.59 effort=1000 velocity=0.5 -> lower=-2.59 upper=0.1 effort=1000 velocity=0.5
- joint motor_front_right_upper_leg: axis 0 -1 0 -> 0 1 0; limit lower=-2.666 upper=1.548 effort=1000 velocity=0.5 -> lower=-1.548 upper=2.666 effort=1000 velocity=0.5
